File: PCB/main/microcontroller_interfacing.kicad_sch (KiCad schematic)
At the start: 11 parts, among them U1 USB_Micro_B_Female_Connector, U2 CH340G, X1 12MHz_SMD_Crystal

Commit message: Update Schematic
Parts:
- C1, C2: footprint (none) -> Footprint_EEE3088F:C0402
- R1: value R -> 82; footprint (none) -> Footprint_EEE3088F:R0603
- R5, R6: footprint (none) -> Footprint_EEE3088F:R0402
- gave numbers to parts that had none: 1
Changed lines of the file:
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@@
     (stroke (width 0) (type default) (color 0 0 0 0))
   )
+  (global_label "+3V3" (shape input) (at 196.85 77.47 90) (fields_autoplaced)
+    (effects (font (size 1.27 1.27)) (justify left))
+    (property "Intersheet References" "${INTERSHEET_REFS}" (id 0) (at 196.7706 69.9769 90)
+      (effects (font (size 1.27 1.27)) (justify left) hide)
+    )
+  )
+  (global_label "+3V3" (shape input) (at 228.6 77.47 90) (fields_autoplaced)
+    (effects (font (size 1.27 1.27)) (justify left))
+    (property "Intersheet References" "${INTERSHEET_REFS}" (id 0) (at 228.5206 69.9769 90)
+      (effects (font (size 1.27 1.27)) (justify left) hide)
+    )
+  )
   (global_label "PF8" (shape input) (at 241.3 103.505 0) (fields_autoplaced)
     (effects (font (size 1.27 1.27)) (justify left))
@@
     )
   )
+  (global_label "+5V" (shape input) (at 91.44 78.74 90) (fields_autoplaced)
+    (effects (font (size 1.27 1.27)) (justify left))
+    (property "Intersheet References" "${INTERSHEET_REFS}" (id 0) (at 91.3606 72.4564 90)
+      (effects (font (size 1.27 1.27)) (justify left) hide)
+    )
+  )
   (global_label "PA9" (shape input) (at 156.21 86.36 0) (fields_autoplaced)
     (effects (font (size 1.27 1.27)) (justify left))
@@
     )
   )
+  (global_label "+3V3" (shape input) (at 121.92 62.23 90) (fields_autoplaced)
+    (effects (font (size 1.27 1.27)) (justify left))
+    (property "Intersheet References" "${INTERSHEET_REFS}" (id 0) (at 121.8406 54.7369 90)
+      (effects (font (size 1.27 1.27)) (justify left) hide)
+    )
+  )
   (symbol (lib_id "Device:C") (at 109.22 133.985 0) (unit 1)
     (in_bom yes) (on_board yes) (fields_autoplaced)
@@
       (effects (font (size 1.27 1.27)) (justify left))
     )
-    (property "Footprint" "" (id 2) (at 110.1852 137.795 0)
+    (property "Footprint" "Footprint_EEE3088F:C0402" (id 2) (at 110.1852 137.795 0)
       (effects (font (size 1.27 1.27)) hide)
     )
@@
     )
     (property "Datasheet" "" (id 3) (at 196.85 114.3 0)
-      (effects (font (size 1.27 1.27)) hide)
-    )
-    (pin "1")
-  )
-  (symbol (lib_id "power:+3V3") (at 228.6 77.47 0) (unit 1)
-    (in_bom yes) (on_board yes) (fields_autoplaced)
-    (property "Reference" "#PWR0103" (id 0) (at 228.6 81.28 0)
-      (effects (font (size 1.27 1.27)) hide)
-    )
-    (property "Value" "+3V3" (id 1) (at 228.6 73.8942 0))
-    (property "Footprint" "" (id 2) (at 228.6 77.47 0)
-      (effects (font (size 1.27 1.27)) hide)
-    )
-    (property "Datasheet" "" (id 3) (at 228.6 77.47 0)
       (effects (font (size 1.27 1.27)) hide)
     )
@@
     (pin "6")
   )
-  (symbol (lib_id "power:+5V") (at 91.44 78.74 0) (unit 1)
-    (in_bom yes) (on_board yes)
-    (property "Reference" "#PWR0112" (id 0) (at 91.44 82.55 0)
-      (effects (font (size 1.27 1.27)) hide)
-    )
-    (property "Value" "+5V" (id 1) (at 91.44 75.1642 0))
-    (property "Footprint" "" (id 2) (at 91.44 78.74 0)
-      (effects (font (size 1.27 1.27)) hide)
-    )
-    (property "Datasheet" "" (id 3) (at 91.44 78.74 0)
-      (effects (font (size 1.27 1.27)) hide)
-    )
-    (pin "1")
-  )
   (symbol (lib_id "power:GND") (at 86.36 107.95 0) (unit 1)
     (in_bom yes) (on_board yes) (fields_autoplaced)
@@
   (symbol (lib_id "Symbol_EEE3088F:AT24C256C-SSHL-T") (at 196.85 103.505 0) (unit 1)
     (in_bom yes) (on_board yes) (fields_autoplaced)
-    (property "Reference" "U?" (id 0) (at 198.8694 94.141 0)
+    (property "Reference" "U3" (id 0) (at 198.8694 94.141 0)
       (effects (font (size 1.27 1.27)) (justify left))
     )
@@
       (effects (font (size 1.27 1.27)) (justify left))
     )
-    (property "Footprint" "" (id 2) (at 233.172 87.63 90)
+    (property "Footprint" "Footprint_EEE3088F:R0402" (id 2) (at 233.172 87.63 90)
       (effects (font (size 1.27 1.27)) hide)
     )
@@
       (effects (font (size 1.27 1.27)) (justify left))
     )
-    (property "Footprint" "" (id 2) (at 220.472 87.63 90)
+    (property "Footprint" "Footprint_EEE3088F:R0402" (id 2) (at 220.472 87.63 90)
       (effects (font (size 1.27 1.27)) hide)
     )
@@
     (pin "2")
   )
-  (symbol (lib_id "power:+3V3") (at 121.92 62.23 0) (unit 1)
-    (in_bom yes) (on_board yes) (fields_autoplaced)
-    (property "Reference" "#PWR0113" (id 0) (at 121.92 66.04 0)
-      (effects (font (size 1.27 1.27)) hide)
-    )
-    (property "Value" "+3V3" (id 1) (at 121.92 58.6542 0))
-    (property "Footprint" "" (id 2) (at 121.92 62.23 0)
-      (effects (font (size 1.27 1.27)) hide)
-    )
-    (property "Datasheet" "" (id 3) (at 121.92 62.23 0)
-      (effects (font (size 1.27 1.27)) hide)
-    )
-    (pin "1")
-  )
   (symbol (lib_id "Device:R") (at 91.44 113.03 0) (unit 1)
     (in_bom yes) (on_board yes) (fields_autoplaced)
@@
       (effects (font (size 1.27 1.27)) (justify left))
     )
-    (property "Value" "R" (id 1) (at 93.218 114.7322 0)
-      (effects (font (size 1.27 1.27)) (justify left))
-    )
-    (property "Footprint" "" (id 2) (at 89.662 113.03 90)
+    (property "Value" "82" (id 1) (at 93.218 114.7322 0)
+      (effects (font (size 1.27 1.27)) (justify left))
+    )
+    (property "Footprint" "Footprint_EEE3088F:R0603" (id 2) (at 89.662 113.03 90)
       (effects (font (size 1.27 1.27)) hide)
     )
@@
       (effects (font (size 1.27 1.27)) (justify left))
     )
-    (property "Footprint" "" (id 2) (at 115.2652 153.67 0)
+    (property "Footprint" "Footprint_EEE3088F:C0402" (id 2) (at 115.2652 153.67 0)
       (effects (font (size 1.27 1.27)) hide)
     )
@@
     (pin "1")
   )
-  (symbol (lib_id "power:+3V3") (at 196.85 77.47 0) (unit 1)
-    (in_bom yes) (on_board yes)
-    (property "Reference" "#PWR0102" (id 0) (at 196.85 81.28 0)
-      (effects (font (size 1.27 1.27)) hide)
-    )
-    (property "Value" "+3V3" (id 1) (at 196.85 73.8942 0))
-    (property "Footprint" "" (id 2) (at 196.85 77.47 0)
-      (effects (font (size 1.27 1.27)) hide)
-    )
-    (property "Datasheet" "" (id 3) (at 196.85 77.47 0)
-      (effects (font (size 1.27 1.27)) hide)
-    )
-    (pin "1")
-  )
   (symbol (lib_id "power:GND") (at 182.88 114.3 0) (unit 1)
     (in_bom yes) (on_board yes) (fields_autoplaced)
-    (property "Reference" "#PWR?" (id 0) (at 182.88 120.65 0)
-      (effects (font (size 1.27 1.27)) hide)
-    )
+    (property "Reference" "#PWR0104" (id 0) (at 182.88 120.65 0)
+      (effects (font (size 1.27 1.27)) hide)
+    )

Commit message: Update Schematic
Connections:
- no-connect marks 0 -> 9
Other:
- title: (none) -> Microcontroller Interfacing
Changed lines of the file:
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@@
 (kicad_sch (version 20211123) (generator eeschema)
   (paper "A4")
+  (title_block
+    (title "Microcontroller Interfacing")
+    (date "2022-03-09")
+    (rev "v1.0")
+  )
   (junction (at 182.88 103.505) (diameter 0) (color 0 0 0 0)
   )
@@
   (junction (at 121.92 68.58) (diameter 0) (color 0 0 0 0)
   )
+  (no_connect (at 134.62 93.98))
+  (no_connect (at 134.62 91.44))
+  (no_connect (at 134.62 104.14))
+  (no_connect (at 134.62 101.6))
+  (no_connect (at 134.62 99.06))
+  (no_connect (at 134.62 96.52))
+  (no_connect (at 114.3 86.36))
+  (no_connect (at 66.04 93.98))
+  (no_connect (at 78.74 96.52))
   (wire (pts (xy 109.22 130.175) (xy 115.57 130.175))
     (stroke (width 0) (type default) (color 0 0 0 0))
