File: PCB/main/outputs.kicad_sch (KiCad schematic)
At the start: 0 parts

Commit message: Add notes
Other:
- company: (none) -> University of Cape Town
Changed lines of the file:
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@@
     (date "2022-03-09")
     (rev "v1.0")
+    (company "University of Cape Town")
+    (comment 4 "Authors: Heather WImberley")
   )
   (text "Not sure if you want this here:\n\nGP LEDS\nPushButton or 2 for testing\nUSB Connector\nTesting Connector\nJumpers for debugging and inserting signals"
