File: PCB/main/Proximity_Sensor.kicad_sch (KiCad schematic)
At the start: 8 parts, among them U6 VL6180XV0NR_1

Commit message: Design PCB
Parts:
- renumbered C8 to C10, C9 to C11, D9 to D7, D10 to D8, R13 to R12, R14 to R13, R15 to R14, U6 to U7
Changed lines of the file:
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@@
   (symbol (lib_id "Device:R") (at 85.09 46.99 0) (unit 1)
     (in_bom yes) (on_board yes) (fields_autoplaced)
-    (property "Reference" "R13" (id 0) (at 87.63 45.7199 0)
+    (property "Reference" "R12" (id 0) (at 87.63 45.7199 0)
       (effects (font (size 1.27 1.27)) (justify left))
     )
@@
   (symbol (lib_id "Device:C_Polarized") (at 151.13 53.34 270) (unit 1)
     (in_bom yes) (on_board yes) (fields_autoplaced)
-    (property "Reference" "C8" (id 0) (at 152.019 45.72 90))
+    (property "Reference" "C10" (id 0) (at 152.019 45.72 90))
     (property "Value" "100nF" (id 1) (at 152.019 48.26 90))
     (property "Footprint" "Capacitor_SMD:C_0402_1005Metric" (id 2) (at 147.32 54.3052 0)
@@
   (symbol (lib_id "power:PWR_FLAG") (at 237.49 22.86 0) (unit 1)
     (in_bom yes) (on_board yes) (fields_autoplaced)
-    (property "Reference" "#FLG04" (id 0) (at 237.49 20.955 0)
+    (property "Reference" "#FLG05" (id 0) (at 237.49 20.955 0)
       (effects (font (size 1.27 1.27)) hide)
     )
@@
   (symbol (lib_id "Device:R") (at 172.72 95.25 0) (unit 1)
     (in_bom yes) (on_board yes) (fields_autoplaced)
-    (property "Reference" "R15" (id 0) (at 175.26 93.9799 0)
+    (property "Reference" "R14" (id 0) (at 175.26 93.9799 0)
       (effects (font (size 1.27 1.27)) (justify left))
     )
@@
   (symbol (lib_id "Device:R") (at 85.09 55.88 0) (unit 1)
     (in_bom yes) (on_board yes) (fields_autoplaced)
-    (property "Reference" "R14" (id 0) (at 87.63 54.6099 0)
+    (property "Reference" "R13" (id 0) (at 87.63 54.6099 0)
       (effects (font (size 1.27 1.27)) (justify left))
     )
@@
   (symbol (lib_id "Device:C_Polarized") (at 151.13 67.31 270) (unit 1)
     (in_bom yes) (on_board yes) (fields_autoplaced)
-    (property "Reference" "C9" (id 0) (at 152.019 59.69 90))
+    (property "Reference" "C11" (id 0) (at 152.019 59.69 90))
     (property "Value" "4.7nF" (id 1) (at 152.019 62.23 90))
     (property "Footprint" "Capacitor_SMD:C_0402_1005Metric" (id 2) (at 147.32 68.2752 0)
@@
   (symbol (lib_id "Diode:BZT52Bxx") (at 85.09 71.12 270) (unit 1)
     (in_bom yes) (on_board yes) (fields_autoplaced)
-    (property "Reference" "D9" (id 0) (at 87.63 69.8499 90)
+    (property "Reference" "D7" (id 0) (at 87.63 69.8499 90)
       (effects (font (size 1.27 1.27)) (justify left))
     )
@@
   (symbol (lib_id "Device:LED") (at 172.72 102.87 90) (unit 1)
     (in_bom yes) (on_board yes) (fields_autoplaced)
-    (property "Reference" "D10" (id 0) (at 176.53 103.1874 90)
+    (property "Reference" "D8" (id 0) (at 176.53 103.1874 90)
       (effects (font (size 1.27 1.27)) (justify right))
     )
@@
   (symbol (lib_id "Symbol_EEE3088F:VL6180XV0NR_1") (at 185.42 59.69 0) (unit 1)
     (in_bom yes) (on_board yes) (fields_autoplaced)
-    (property "Reference" "U6" (id 0) (at 210.82 52.07 0))
+    (property "Reference" "U7" (id 0) (at 210.82 52.07 0))
     (property "Value" "VL6180XV0NR_1" (id 1) (at 210.82 54.61 0))
     (property "Footprint" "Footprint_EEE3088F:LGA-12_L4.8-W2.8-P0.75-BL" (id 2) (at 185.42 49.53 0)
