File: PCB/main/Cutout_protection.kicad_sch (KiCad schematic)
At the start: 8 parts, among them K1 ADW11, Q3 2N3904, U2 LM358DR2G

Commit message: Design PCB
Parts:
- added TP4: TestPoint, TestPoint:TestPoint_Pad_D1.0mm, symbol Connector:TestPoint
- renumbered D4 to D5, D5 to D6, Q3 to Q2, R4 to R10, R5 to R11, R3 to R9, U2 to U6
Connections:
- net Relay_OUT: now also TP4.1
Changed lines of the file:
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@@
   (junction (at 82.55 120.65) (diameter 0) (color 0 0 0 0)
+  )
+  (junction (at 169.545 101.6) (diameter 0) (color 0 0 0 0)
   )
   (junction (at 130.81 101.6) (diameter 0) (color 0 0 0 0)
@@
     (stroke (width 0) (type default) (color 0 0 0 0))
   )
+  (wire (pts (xy 169.545 101.6) (xy 179.07 101.6))
+    (stroke (width 0) (type default) (color 0 0 0 0))
+  )
   (wire (pts (xy 54.61 120.65) (xy 59.69 120.65))
     (stroke (width 0) (type default) (color 0 0 0 0))
@@
     (stroke (width 0) (type default) (color 0 0 0 0))
   )
-  (wire (pts (xy 160.02 101.6) (xy 179.07 101.6))
+  (wire (pts (xy 160.02 101.6) (xy 169.545 101.6))
     (stroke (width 0) (type default) (color 0 0 0 0))
   )
@@
   (symbol (lib_id "Simulation_SPICE:DIODE") (at 130.81 93.98 90) (unit 1)
     (in_bom yes) (on_board yes) (fields_autoplaced)
-    (property "Reference" "D5" (id 0) (at 133.35 92.7099 90)
+    (property "Reference" "D6" (id 0) (at 133.35 92.7099 90)
       (effects (font (size 1.27 1.27)) (justify right))
     )
@@
   (symbol (lib_id "Device:R") (at 59.69 93.98 0) (unit 1)
     (in_bom yes) (on_board yes) (fields_autoplaced)
-    (property "Reference" "R3" (id 0) (at 62.23 92.7099 0)
+    (property "Reference" "R9" (id 0) (at 62.23 92.7099 0)
       (effects (font (size 1.27 1.27)) (justify left))
     )
@@
   (symbol (lib_id "Transistor_BJT:2N3904") (at 128.27 110.49 0) (unit 1)
     (in_bom yes) (on_board yes) (fields_autoplaced)
-    (property "Reference" "Q3" (id 0) (at 133.35 109.2199 0)
+    (property "Reference" "Q2" (id 0) (at 133.35 109.2199 0)
       (effects (font (size 1.27 1.27)) (justify left))
     )
@@
   (symbol (lib_id "power:GND") (at 54.61 127 0) (unit 1)
     (in_bom yes) (on_board yes) (fields_autoplaced)
-    (property "Reference" "#PWR018" (id 0) (at 54.61 133.35 0)
+    (property "Reference" "#PWR034" (id 0) (at 54.61 133.35 0)
       (effects (font (size 1.27 1.27)) hide)
     )
@@
   (symbol (lib_id "Device:R") (at 82.55 93.98 0) (unit 1)
     (in_bom yes) (on_board yes) (fields_autoplaced)
-    (property "Reference" "R4" (id 0) (at 85.09 92.7099 0)
+    (property "Reference" "R10" (id 0) (at 85.09 92.7099 0)
       (effects (font (size 1.27 1.27)) (justify left))
     )
@@
     (pin "2")
   )
+  (symbol (lib_id "Connector:TestPoint") (at 169.545 101.6 180) (unit 1)
+    (in_bom yes) (on_board yes) (fields_autoplaced)
+    (property "Reference" "TP4" (id 0) (at 170.942 104.0673 0)
+      (effects (font (size 1.27 1.27)) (justify right))
+    )
+    (property "Value" "TestPoint" (id 1) (at 170.942 106.6042 0)
+      (effects (font (size 1.27 1.27)) (justify right))
+    )
+    (property "Footprint" "TestPoint:TestPoint_Pad_D1.0mm" (id 2) (at 164.465 101.6 0)
+      (effects (font (size 1.27 1.27)) hide)
+    )
+    (property "Datasheet" "~" (id 3) (at 164.465 101.6 0)
+      (effects (font (size 1.27 1.27)) hide)
+    )
+    (pin "1")
+  )
   (symbol (lib_id "Device:R") (at 82.55 111.76 0) (unit 1)
     (in_bom yes) (on_board yes) (fields_autoplaced)
-    (property "Reference" "R5" (id 0) (at 85.09 110.4899 0)
+    (property "Reference" "R11" (id 0) (at 85.09 110.4899 0)
       (effects (font (size 1.27 1.27)) (justify left))
     )
@@
   (symbol (lib_id "Symbol_EEE3088F:LM358DR2G") (at 106.68 101.6 0) (unit 1)
     (in_bom yes) (on_board yes) (fields_autoplaced)
-    (property "Reference" "U2" (id 0) (at 116.84 96.901 0))
+    (property "Reference" "U6" (id 0) (at 116.84 96.901 0))
     (property "Value" "LM358DR2G" (id 1) (at 116.84 99.441 0))
     (property "Footprint" "Package_SO:SOIC-8_3.9x4.9mm_P1.27mm" (id 2) (at 106.68 101.6 0)
@@
   (symbol (lib_id "power:PWR_FLAG") (at 66.675 43.18 0) (unit 1)
     (in_bom yes) (on_board yes) (fields_autoplaced)
-    (property "Reference" "#FLG0102" (id 0) (at 66.675 41.275 0)
+    (property "Reference" "#FLG04" (id 0) (at 66.675 41.275 0)
       (effects (font (size 1.27 1.27)) hide)
     )
@@
   (symbol (lib_id "Device:D_Zener") (at 59.69 111.76 270) (unit 1)
     (in_bom yes) (on_board yes) (fields_autoplaced)
-    (property "Reference" "D4" (id 0) (at 62.23 110.4899 90)
-      (effects (font (size 1.27 1.27)) (justify left))
-    )
+    (property "Reference" "D5" (id 0) (at 62.23 110.4899 90)
+      (effects (font (size 1.27 1.27)) (justify left))
+    )

Commit message: Change names
Parts:
- K1: value ADW11 -> G5NB
- Q2: value 2N3904 -> MMBT3904
Changed lines of the file:
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@@
   (symbol (lib_id "Transistor_BJT:2N3904") (at 128.27 110.49 0) (unit 1)
     (in_bom yes) (on_board yes) (fields_autoplaced)
-    (property "Reference" "Q2" (id 0) (at 133.35 109.2199 0)
+    (property "Reference" "Q2" (id 0) (at 133.1214 109.6553 0)
       (effects (font (size 1.27 1.27)) (justify left))
     )
-    (property "Value" "2N3904" (id 1) (at 133.35 111.7599 0)
+    (property "Value" "MMBT3904" (id 1) (at 133.1214 112.1922 0)
       (effects (font (size 1.27 1.27)) (justify left))
     )
@@
   (symbol (lib_id "Relay:G5Q-1A") (at 154.94 93.98 0) (unit 1)
     (in_bom yes) (on_board yes) (fields_autoplaced)
-    (property "Reference" "K1" (id 0) (at 166.37 92.7099 0)
+    (property "Reference" "K1" (id 0) (at 163.322 93.1453 0)
       (effects (font (size 1.27 1.27)) (justify left))
     )
-    (property "Value" "ADW11" (id 1) (at 166.37 95.2499 0)
+    (property "Value" "G5NB" (id 1) (at 163.322 95.6822 0)
       (effects (font (size 1.27 1.27)) (justify left))
     )
