File: PCB/main/Cutout_protection.kicad_sch (KiCad schematic)
At the start: 9 parts, among them K1 G5NB, Q2 MMBT3904, U6 LM358DR2G

Commit message: Revert "again"
This reverts commit 3983b3a2bbd3cb989ba3f9e8c32b60b336cbf8a7
Parts:
- TP4: value CutP -> TestPoint
Changed lines of the file:
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@@
   (symbol (lib_id "Connector:TestPoint") (at 169.545 101.6 180) (unit 1)
     (in_bom yes) (on_board yes) (fields_autoplaced)
-    (property "Reference" "TP4" (id 0) (at 171.45 103.6319 0)
+    (property "Reference" "TP4" (id 0) (at 170.942 104.0673 0)
       (effects (font (size 1.27 1.27)) (justify right))
     )
-    (property "Value" "CutP" (id 1) (at 171.45 106.1719 0)
+    (property "Value" "TestPoint" (id 1) (at 170.942 106.6042 0)
       (effects (font (size 1.27 1.27)) (justify right))
     )
@@
   (symbol (lib_id "power:PWR_FLAG") (at 66.675 43.18 0) (unit 1)
     (in_bom yes) (on_board yes) (fields_autoplaced)
-    (property "Reference" "#FLG03" (id 0) (at 66.675 41.275 0)
+    (property "Reference" "#FLG04" (id 0) (at 66.675 41.275 0)
       (effects (font (size 1.27 1.27)) hide)
     )
