File: PCB/main/temperature_sensor.kicad_sch (KiCad schematic)
At the start: 6 parts, among them Q1 FDS6690A, U7 MCP9700T-ETT

Commit message: Design PCB
Parts:
- added TP5, TP6: TestPoint, TestPoint:TestPoint_Pad_D1.0mm, symbol Connector:TestPoint
- renumbered D11 to D9, Q1 to Q3, R16 to R15, R17 to R16, R18 to R17, U7 to U8
Connections:
- net Output: now also TP6.1
- net Vdd: now also TP5.1
Changed lines of the file:
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@@
   (junction (at 146.05 63.5) (diameter 0) (color 0 0 0 0)
+  )
+  (junction (at 150.495 66.04) (diameter 0) (color 0 0 0 0)
+  )
+  (junction (at 206.375 74.93) (diameter 0) (color 0 0 0 0)
   )
   (no_connect (at 112.395 81.28))
@@
     (stroke (width 0) (type default) (color 0 0 0 0))
   )
+  (wire (pts (xy 150.495 66.04) (xy 165.1 66.04))
+    (stroke (width 0) (type default) (color 0 0 0 0))
+  )
   (wire (pts (xy 165.1 82.55) (xy 165.1 135.89))
     (stroke (width 0) (type default) (color 0 0 0 0))
@@
     (stroke (width 0) (type default) (color 0 0 0 0))
   )
-  (wire (pts (xy 186.69 74.93) (xy 218.44 74.93))
+  (wire (pts (xy 186.69 74.93) (xy 206.375 74.93))
     (stroke (width 0) (type default) (color 0 0 0 0))
   )
@@
     (stroke (width 0) (type default) (color 0 0 0 0))
   )
+  (wire (pts (xy 206.375 74.93) (xy 218.44 74.93))
+    (stroke (width 0) (type default) (color 0 0 0 0))
+  )
   (wire (pts (xy 109.855 63.5) (xy 109.855 66.04))
     (stroke (width 0) (type default) (color 0 0 0 0))
@@
     (stroke (width 0) (type default) (color 0 0 0 0))
   )
-  (wire (pts (xy 146.05 66.04) (xy 165.1 66.04))
+  (wire (pts (xy 146.05 66.04) (xy 150.495 66.04))
     (stroke (width 0) (type default) (color 0 0 0 0))
   )
@@
   (symbol (lib_id "Device:R") (at 186.69 86.36 0) (unit 1)
     (in_bom yes) (on_board yes) (fields_autoplaced)
-    (property "Reference" "R18" (id 0) (at 189.23 85.0899 0)
+    (property "Reference" "R17" (id 0) (at 189.23 85.0899 0)
       (effects (font (size 1.27 1.27)) (justify left))
     )
@@
   (symbol (lib_id "Device:LED") (at 186.69 99.06 90) (unit 1)
     (in_bom yes) (on_board yes) (fields_autoplaced)
-    (property "Reference" "D11" (id 0) (at 190.5 99.3774 90)
+    (property "Reference" "D9" (id 0) (at 190.5 99.3774 90)
       (effects (font (size 1.27 1.27)) (justify right))
     )
@@
   (symbol (lib_id "Sensor_Temperature:MCP9700T-ETT") (at 165.1 74.93 0) (unit 1)
     (in_bom yes) (on_board yes) (fields_autoplaced)
-    (property "Reference" "U7" (id 0) (at 156.21 73.6599 0)
+    (property "Reference" "U8" (id 0) (at 156.21 73.6599 0)
       (effects (font (size 1.27 1.27)) (justify right))
     )
@@
   (symbol (lib_id "Device:R") (at 146.05 41.91 0) (unit 1)
     (in_bom yes) (on_board yes) (fields_autoplaced)
-    (property "Reference" "R16" (id 0) (at 148.59 40.6399 0)
+    (property "Reference" "R15" (id 0) (at 148.59 40.6399 0)
       (effects (font (size 1.27 1.27)) (justify left))
     )
@@
   (symbol (lib_id "Device:R") (at 146.05 53.34 0) (unit 1)
     (in_bom yes) (on_board yes) (fields_autoplaced)
-    (property "Reference" "R17" (id 0) (at 148.59 52.0699 0)
+    (property "Reference" "R16" (id 0) (at 148.59 52.0699 0)
       (effects (font (size 1.27 1.27)) (justify left))
     )
@@
     (pin "2")
   )
+  (symbol (lib_id "Connector:TestPoint") (at 150.495 66.04 0) (unit 1)
+    (in_bom yes) (on_board yes) (fields_autoplaced)
+    (property "Reference" "TP5" (id 0) (at 151.892 61.9033 0)
+      (effects (font (size 1.27 1.27)) (justify left))
+    )
+    (property "Value" "TestPoint" (id 1) (at 151.892 64.4402 0)
+      (effects (font (size 1.27 1.27)) (justify left))
+    )
+    (property "Footprint" "TestPoint:TestPoint_Pad_D1.0mm" (id 2) (at 155.575 66.04 0)
+      (effects (font (size 1.27 1.27)) hide)
+    )
+    (property "Datasheet" "~" (id 3) (at 155.575 66.04 0)
+      (effects (font (size 1.27 1.27)) hide)
+    )
+    (pin "1")
+  )
   (symbol (lib_id "power:GND") (at 92.71 135.89 270) (unit 1)
     (in_bom yes) (on_board yes) (fields_autoplaced)
@@
   (symbol (lib_id "Symbol_EEE3088F:FDS6690A") (at 102.235 73.66 0) (unit 1)
     (in_bom yes) (on_board yes) (fields_autoplaced)
-    (property "Reference" "Q1" (id 0) (at 118.745 72.3899 0)
+    (property "Reference" "Q3" (id 0) (at 118.745 72.3899 0)
       (effects (font (size 1.27 1.27)) (justify left))
     )
@@
     (pin "8")
   )
+  (symbol (lib_id "Connector:TestPoint") (at 206.375 74.93 0) (unit 1)
+    (in_bom yes) (on_board yes) (fields_autoplaced)
+    (property "Reference" "TP6" (id 0) (at 207.772 70.7933 0)
+      (effects (font (size 1.27 1.27)) (justify left))
+    )
+    (property "Value" "TestPoint" (id 1) (at 207.772 73.3302 0)
+      (effects (font (size 1.27 1.27)) (justify left))
+    )
+    (property "Footprint" "TestPoint:TestPoint_Pad_D1.0mm" (id 2) (at 211.455 74.93 0)
+      (effects (font (size 1.27 1.27)) hide)
+    )
+    (property "Datasheet" "~" (id 3) (at 211.455 74.93 0)
+      (effects (font (size 1.27 1.27)) hide)
+    )
+    (pin "1")
+  )
 )
