File: PCB/temperature_sensor.kicad_sch (KiCad schematic)
At the start: 8 parts, among them Q3 FDS6690A, U8 MCP9700T-ETT

Commit message: pcb revive
Parts:
- TP5: value TestPoint -> TempVcc
- TP6: value TestPoint -> TempOut
Changed lines of the file:
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@@
   (symbol (lib_id "power:PWR_FLAG") (at 213.995 32.385 0) (unit 1)
     (in_bom yes) (on_board yes) (fields_autoplaced)
-    (property "Reference" "#FLG06" (id 0) (at 213.995 30.48 0)
+    (property "Reference" "#FLG05" (id 0) (at 213.995 30.48 0)
       (effects (font (size 1.27 1.27)) hide)
     )
@@
   (symbol (lib_id "Connector:TestPoint") (at 150.495 66.04 0) (unit 1)
     (in_bom yes) (on_board yes) (fields_autoplaced)
-    (property "Reference" "TP5" (id 0) (at 151.892 61.9033 0)
+    (property "Reference" "TP5" (id 0) (at 152.4 61.4679 0)
       (effects (font (size 1.27 1.27)) (justify left))
     )
-    (property "Value" "TestPoint" (id 1) (at 151.892 64.4402 0)
+    (property "Value" "TempVcc" (id 1) (at 152.4 64.0079 0)
       (effects (font (size 1.27 1.27)) (justify left))
     )
@@
   (symbol (lib_id "Connector:TestPoint") (at 206.375 74.93 0) (unit 1)
     (in_bom yes) (on_board yes) (fields_autoplaced)
-    (property "Reference" "TP6" (id 0) (at 207.772 70.7933 0)
+    (property "Reference" "TP6" (id 0) (at 208.28 70.3579 0)
       (effects (font (size 1.27 1.27)) (justify left))
     )
-    (property "Value" "TestPoint" (id 1) (at 207.772 73.3302 0)
+    (property "Value" "TempOut" (id 1) (at 208.28 72.8979 0)
       (effects (font (size 1.27 1.27)) (justify left))
     )
