File: PCB/power.kicad_sch (KiCad schematic)
At the start: 22 parts, among them Q1 AO3401A, U1 LP2951-33DR, U2 AMS1117

Commit message: pcb revive
Parts:
- TP1: value TestPoint -> BatPP
- TP2: value TestPoint -> 3.3V
Changed lines of the file:
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@@
   (symbol (lib_id "Connector:TestPoint") (at 242.57 126.365 0) (unit 1)
     (in_bom yes) (on_board yes) (fields_autoplaced)
-    (property "Reference" "TP2" (id 0) (at 243.967 122.2283 0)
-      (effects (font (size 1.27 1.27)) (justify left))
-    )
-    (property "Value" "TestPoint" (id 1) (at 243.967 124.7652 0)
+    (property "Reference" "TP2" (id 0) (at 245.11 121.7929 0)
+      (effects (font (size 1.27 1.27)) (justify left))
+    )
+    (property "Value" "3.3V" (id 1) (at 245.11 124.3329 0)
       (effects (font (size 1.27 1.27)) (justify left))
     )
@@
   (symbol (lib_id "Connector:TestPoint") (at 73.025 66.04 180) (unit 1)
     (in_bom yes) (on_board yes) (fields_autoplaced)
-    (property "Reference" "TP1" (id 0) (at 74.422 68.5073 0)
+    (property "Reference" "TP1" (id 0) (at 74.93 68.0719 0)
       (effects (font (size 1.27 1.27)) (justify right))
     )
-    (property "Value" "TestPoint" (id 1) (at 74.422 71.0442 0)
+    (property "Value" "BatPP" (id 1) (at 74.93 70.6119 0)
       (effects (font (size 1.27 1.27)) (justify right))
     )

Commit message: POWER CHANGES YAAASSSSSSS
Parts:
- removed C1: 0.1uF, Capacitor_SMD:C_0402_1005Metric, symbol Device:C
- removed C2: 22uF, Capacitor_SMD:C_0603_1608Metric, symbol Device:C
- removed C3: 330pF, Capacitor_SMD:C_0402_1005Metric, symbol Device:C
- removed C5: 100uF, Capacitor_SMD:C_1206_3216Metric, symbol Device:C_Polarized
- removed D2: DIODE, Footprint_EEE3088F:DO-214AC_L4.3-W2.7-LS5.3-RD, symbol Simulation_SPICE:DIODE
- removed JP1: SolderJumper_2_Bridged, Jumper:SolderJumper-2_P1.3mm_Bridged2Bar_Pad1.0x1.5mm, symbol Jumper:SolderJumper_2_Bridged
- removed R2: 2M, Resistor_SMD:R_0805_2012Metric, symbol Device:R
- removed R3: 806K, Resistor_SMD:R_0402_1005Metric, symbol Device:R
- removed RV1: 50K, Footprint_EEE3088F:VG039NCHXTB503, symbol Device:R_Potentiometer
- removed U1: LP2951-33DR, Package_SO:SOIC-8_3.9x4.9mm_P1.27mm, symbol Regulator_Linear:LP2951-3.3_DIP
- removed U2: AMS1117, Package_TO_SOT_SMD:SOT-223-3_TabPin2, symbol Regulator_Linear:AMS1117
- added C?: 1uF, Capacitor_SMD:C_0402_1005Metric, symbol Device:C
- added C?: 0.1uF, symbol Device:C_Small
- added C? (x2): 10uF, symbol Device:C_Small
- added D?: RLED, symbol Device:LED
- added D?: GLED, symbol Device:LED
- added Q? (x2): 2N7002, Package_TO_SOT_SMD:SOT-23, symbol Transistor_FET:2N7002
- added R?: 100, symbol Device:R
- added R? (x3): 1k, symbol Device:R
- added R?: 1.2k, symbol Device:R
- added R?: 0.4, symbol Device:R
- added U?: FS312F-G, symbol Battery_Management:FS312F-G
- added U?: TP4056, symbol Battery_Management:TP4056
- added U?: XC6206P332MR, Package_TO_SOT_SMD:SOT-23, symbol Regulator_Linear:XC6206PxxxMR
- C4: value 0.1uF -> 1uF
Connections:
- net Relay_OUT is gone; now on net +5V (REVERSE PROTECTED): JP4.1 (A)
- net +3.3V: now also C?.1, U?.2 (VO)
- net +5V (INPUT PROTECTED): now also R?.1
- net +5V (protected_jumped): now also U?.3 (VI)
- net Battery +: now also C?.1, R?.1, U?.5 (BAT)
- net GND: now also C?.2, C?.2, C?.2, Q?.2 (S), R?.2, R?.2, U?.1 (GND), U?.1 (TEMP), U?.3 (GND), U?.9 (EP); no longer BT1.2 (-)
- new net: BT1.2 (-), C?.1, Q?.2 (S), U?.6 (GND)
- new net: C?.2, R?.2, U?.5 (Vcc)
- new net: Q?.1 (G), U?.1 (OD)
- new net: R?.1, U?.2 (CS)
- new net: Q?.1 (G), U?.3 (OC)
- new net: D?.1 (K), R?.1 (x2)
- new net: C?.1, D?.2 (A), D?.2 (A), R?.2, U?.4 (Vcc), U?.8 (CE)
- new net: R?.1, U?.2 (PROG)
- new net: R?.2, U?.6 (STDBY)
- new net: R?.2, U?.7 (CHRG)
- new net: Q?.3 (D), Q?.3 (D)
- no-connect marks 3 -> 1
Other:
- removed sheet Cutout Proctection
- note removed: "Battery Connection"
- moved on the sheet: BT1, D1, JP3, TP1

Commit message: Prepare PCB
Parts:
- C1, C2: renamed from C?; footprint (none) -> Capacitor_SMD:C_0402_1005Metric; JLC Part # (none) -> C15525; LCSC (none) -> C15525
- C3: renamed from C?; value 0.1uF -> 100nF; footprint (none) -> Capacitor_SMD:C_0402_1005Metric; JLC Part # (none) -> C1525; LCSC (none) -> C1525
- C4: JLC Part # C1525 -> C52923; LCSC (none) -> C52923
- C5: renamed from C?; JLC Part # C1525 -> C52923; LCSC (none) -> C52923
- D1: LCSC (none) -> C408389
- D2: renamed from D?; value GLED -> YLED; footprint (none) -> LED_SMD:LED_0805_2012Metric; JLC Part # (none) -> C2296; LCSC (none) -> C2296
- D3: LCSC (none) -> C8061
- D6: renamed from D?; footprint (none) -> LED_SMD:LED_0603_1608Metric; JLC Part # (none) -> C2286; LCSC (none) -> C2286
- Q1: LCSC (none) -> C15127
- Q2, Q3: renamed from Q?; value 2N7002 -> AO3401A; JLC Part # (none) -> C15127; LCSC (none) -> C15127
- R1: LCSC (none) -> C22775
- R13, R3, R7: renamed from R?; footprint (none) -> Resistor_SMD:R_0603_1608Metric; JLC Part # (none) -> C21190; LCSC (none) -> C21190
- R2: renamed from R?; footprint (none) -> Resistor_SMD:R_0805_2012Metric; JLC Part # (none) -> C52548; LCSC (none) -> C52548
- R8: renamed from R?; footprint (none) -> Resistor_SMD:R_0603_1608Metric; JLC Part # (none) -> C22765; LCSC (none) -> C22765
- R9: renamed from R?; footprint (none) -> Resistor_SMD:R_0603_1608Metric; JLC Part # (none) -> C22775; LCSC (none) -> C22775
- U1: renamed from U?; footprint (none) -> Footprint_EEE3088F:ESOP-8_L4.9-W3.9-P1.27-LS6.0-BL-EP; JLC Part # (none) -> C16581; LCSC (none) -> C16581
- U2: renamed from U?; footprint (none) -> Package_TO_SOT_SMD:SOT-23-6; JLC Part # (none) -> C82736; LCSC (none) -> C82736
- U6: renamed from U?; LCSC (none) -> C5446

Commit message: Final Schematic changes
Parts:
- Q2, Q3: value AO3401A -> 2N7002; JLC Part # C15127 -> C8545; LCSC C15127 -> C8545
Changed lines of the file:
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@@
     (in_bom yes) (on_board yes) (fields_autoplaced)
     (property "Reference" "Q3" (id 0) (at 227.33 80.1354 90))
-    (property "Value" "AO3401A" (id 1) (at 227.33 82.6723 90))
+    (property "Value" "2N7002" (id 1) (at 227.33 82.6723 90))
     (property "Footprint" "Package_TO_SOT_SMD:SOT-23" (id 2) (at 229.235 78.74 0)
       (effects (font (size 1.27 1.27) italic) (justify left) hide)
@@
       (effects (font (size 1.27 1.27)) (justify left) hide)
     )
-    (property "JLC Part #" "C15127" (id 4) (at 227.33 73.66 0)
-      (effects (font (size 1.27 1.27)) hide)
-    )
-    (property "LCSC" "C15127" (id 5) (at 227.33 73.66 0)
+    (property "JLC Part #" "C8545" (id 4) (at 227.33 73.66 0)
+      (effects (font (size 1.27 1.27)) hide)
+    )
+    (property "LCSC" "C8545" (id 5) (at 227.33 73.66 0)
       (effects (font (size 1.27 1.27)) hide)
     )
@@
     (in_bom yes) (on_board yes) (fields_autoplaced)
     (property "Reference" "Q2" (id 0) (at 212.09 80.1354 90))
-    (property "Value" "AO3401A" (id 1) (at 212.09 82.6723 90))
+    (property "Value" "2N7002" (id 1) (at 212.09 82.6723 90))
     (property "Footprint" "Package_TO_SOT_SMD:SOT-23" (id 2) (at 210.185 78.74 0)
       (effects (font (size 1.27 1.27) italic) (justify left) hide)
@@
       (effects (font (size 1.27 1.27)) (justify left) hide)
     )
-    (property "JLC Part #" "C15127" (id 4) (at 212.09 73.66 0)
-      (effects (font (size 1.27 1.27)) hide)
-    )
-    (property "LCSC" "C15127" (id 5) (at 212.09 73.66 0)
-      (effects (font (size 1.27 1.27)) hide)
-    )
+    (property "JLC Part #" "C8545" (id 4) (at 212.09 73.66 0)
+      (effects (font (size 1.27 1.27)) hide)
+    )
+    (property "LCSC" "C8545" (id 5) (at 212.09 73.66 0)
+      (effects (font (size 1.27 1.27)) hide)
+    )
