File: PCB/main.kicad_pcb (KiCad board)
At the start: 2 copper layers, 100 x 100 mm, 74 parts, among them J1 Conn_01x10_Male, J2 Conn_01x33_Female, J3 Conn_01x33_Female, J4 Conn_01x33_Female, J5 Conn_01x33_Female, K1 G5NB, Q1 AO3401A, Q2 MMBT3904, Q3 FDS6690A, U1 LP2951-33DR, U2 AMS1117, U3 CH340G, U4 USB_Micro_B, U5 AT24C256C-SSHL-T, U6 LM358DR2G, U7 VL6180XV0NR_1, U8 MCP9700T-ETT, X1 12MHz Crystal

Commit message: Prepare PCB
Parts:
- removed D7: BZT52C3V0, Diode_SMD:D_SOD-123
- removed JP1, JP10: SolderJumper_2_Bridged, Jumper:SolderJumper-2_P1.3mm_Bridged2Bar_Pad1.0x1.5mm
- removed K1: G5NB, Relay_THT:Relay_SPST_Omron-G5Q-1A
- removed R14, R17: 10k, Resistor_SMD:R_0402_1005Metric
- removed R15: 330, Resistor_SMD:R_0402_1005Metric
- removed R16: 220, Resistor_SMD:R_0402_1005Metric
- removed RV1: 50K, Footprint_EEE3088F:VG039NCHXTB503
- removed TP4: CutP, TestPoint:TestPoint_Pad_D1.0mm
- removed TP6: TempOut, TestPoint:TestPoint_Pad_D1.0mm
- added C12: 1uF, Capacitor_SMD:C_0402_1005Metric, F.Cu at (79.0, 108.4)
- C1: value 0.1uF -> 10uF
- C2: value 22uF -> 10uF; footprint Capacitor_SMD:C_0603_1608Metric -> Capacitor_SMD:C_0402_1005Metric
- C3: value 330pF -> 100nF
- C4: value 0.1uF -> 1uF
- C5: value 100uF -> 1uF; footprint Capacitor_SMD:C_1206_3216Metric -> Capacitor_SMD:C_0402_1005Metric
- C9: value 0.1uF -> 100nF
- D2: value DIODE -> YLED; footprint Footprint_EEE3088F:DO-214AC_L4.3-W2.7-LS5.3-RD -> LED_SMD:LED_0805_2012Metric
- D4, D9: value LED -> RLED
- D5: value ZMM4V7-M -> DIODE; footprint Footprint_EEE3088F:LL-34_L3.5-W1.5-RD -> Footprint_EEE3088F:DO-214AC_L4.3-W2.7-LS5.3-RD
- D6: value DIODE -> RLED; footprint Footprint_EEE3088F:DO-214AC_L4.3-W2.7-LS5.3-RD -> LED_SMD:LED_0603_1608Metric
- D8: value LED -> BZT52C3V0; footprint LED_SMD:LED_0603_1608Metric -> Diode_SMD:D_SOD-123
- Q2: value MMBT3904 -> AO3401A
- Q3: value FDS6690A -> AO3401A; footprint Package_SO:SOIC-8_3.9x4.9mm_P1.27mm -> Package_TO_SOT_SMD:SOT-23
- R10: value 1k -> 330
- R11: value 100k -> 10k
- R13: value 330 -> 1k; footprint Resistor_SMD:R_0402_1005Metric -> Resistor_SMD:R_0603_1608Metric
- R2: value 2M -> 0.4
- R3: value 806K -> 1k; footprint Resistor_SMD:R_0402_1005Metric -> Resistor_SMD:R_0603_1608Metric
- R4: value 2.7k -> 150
- R5: value 4.7k -> 10k
- R6: value 82 -> 10k; footprint Resistor_SMD:R_0603_1608Metric -> Resistor_SMD:R_0402_1005Metric
- R7: value 10k -> 1k; footprint Resistor_SMD:R_0402_1005Metric -> Resistor_SMD:R_0603_1608Metric
- R8: value 10k -> 1.2k; footprint Resistor_SMD:R_0402_1005Metric -> Resistor_SMD:R_0603_1608Metric
- R9: value 150 -> 100; footprint Resistor_SMD:R_0402_1005Metric -> Resistor_SMD:R_0603_1608Metric
- TP5: value TempVcc -> TempOut
- U1: value LP2951-33DR -> TP4056; footprint Package_SO:SOIC-8_3.9x4.9mm_P1.27mm -> Footprint_EEE3088F:ESOP-8_L4.9-W3.9-P1.27-LS6.0-BL-EP
- U2: value AMS1117 -> FS312F-G; footprint Package_TO_SOT_SMD:SOT-223-3_TabPin2 -> Package_TO_SOT_SMD:SOT-23-6
- U6: value LM358DR2G -> XC6206P332MR; footprint Package_SO:SOIC-8_3.9x4.9mm_P1.27mm -> Package_TO_SOT_SMD:SOT-23
- moved Q3 107.7 mm to (207.3, 134.2)
- moved U2 80.1 mm to (198.1, 122.4), turned to 0 degrees
- moved G*** 77.7 mm to (199.9, 58.8)
- moved C8 76.5 mm to (225.8, 97.8)
- moved C6 73.0 mm to (224.1, 92.2)
- moved X1 71.6 mm to (223.0, 82.5)
- moved TP2 70.1 mm to (223.8, 104.8)
- moved JP4 67.4 mm to (200.4, 147.7), turned to -90 degrees
- moved C5 66.1 mm to (196.5, 143.2)
- moved C7 61.1 mm to (219.0, 88.3)
- moved U5 60.6 mm to (207.6, 95.6)
- moved R7 59.8 mm to (213.8, 111.0)
- moved R8 59.7 mm to (213.8, 115.6)
- moved C4 59.0 mm to (191.2, 146.9)
- moved U3 56.6 mm to (214.4, 78.4)
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Connections:
- BT1 pad 2: GND -> Net-(BT1-Pad2)
- C1 pad 1: /Power/+5V jumped -> Net-(C1-Pad1)
- C10 pad 1: /Sensing/Proximity_Sensor/VCC -> Net-(C10-Pad1)
- C11 pad 1: /Sensing/Proximity_Sensor/VCC -> Net-(C10-Pad1)
- C2 pad 1: Net-(C2-Pad1) -> /Power/Battery +
- C3 pad 1: /Power/Battery + -> Net-(BT1-Pad2)
- C7 pad 1: /microcontroller_interfacing/+5V -> Net-(C7-Pad1)
- D2 pad 1: Net-(C2-Pad1) -> Net-(D2-Pad1)
- D2 pad 2: /Power/Battery + -> Net-(C1-Pad1)
- D4 pad 1: Net-(D4-Pad1) -> /PA4
- D4 pad 2: /microcontroller_interfacing/+5V -> /microcontroller_interfacing/USB_Detect
- D5 pad 1: Net-(D5-Pad1) -> /microcontroller_interfacing/USB_Detect
- D5 pad 2: GND -> /microcontroller_interfacing/+5V
- D6 pad 2: /Power/Battery + -> Net-(C1-Pad1)
- D8 pad 1: GND -> Net-(C10-Pad1)
- D8 pad 2: Net-(D8-Pad2) -> GND
- JP4 pad 1: /Power/Relay_OUT -> /Power/+5V (REVERSE PROTECTED)
- JP5 pad 2: /Sensing/Temperature_Sensor/3.3V -> /Sensing/Proximity_Sensor/VCC
- JP6 pad 1: VDD -> /microcontroller_interfacing/D+
- JP6 pad 2: /Sensing/Proximity_Sensor/VCC -> Net-(JP6-Pad2)
- JP7 pad 1: /microcontroller_interfacing/D+ -> /microcontroller_interfacing/D-
- JP8 pad 1: /microcontroller_interfacing/D- -> Net-(JP8-Pad1)
- JP8 pad 2: Net-(JP8-Pad2) -> /PB7
- JP9 pad 2: /PB7 -> /PB8
- Q2 pad 1: GND -> Net-(Q2-Pad1)
- Q2 pad 2: Net-(Q2-Pad2) -> Net-(BT1-Pad2)
- Q2 pad 3: Net-(D6-Pad1) -> Net-(Q2-Pad3)
- Q3 pad 1: GND -> Net-(Q3-Pad1)
- Q3 pad 2: unconnected-(Q3-Pad2) -> GND
- Q3 pad 3: unconnected-(Q3-Pad3) -> Net-(Q2-Pad3)
- R10 pad 1: /Power/Battery + -> /Sensing/Proximity_Sensor/VCC
- R10 pad 2: Net-(R10-Pad2) -> Net-(C10-Pad1)
- R11 pad 1: Net-(R10-Pad2) -> /PB4
- R11 pad 2: GND -> Net-(D9-Pad2)
- R12 pad 1: /Sensing/Proximity_Sensor/VCC -> /PB0
- R12 pad 2: Net-(R12-Pad2) -> Net-(C12-Pad1)
- R13 pad 1: Net-(R12-Pad2) -> Net-(R13-Pad1)
- R13 pad 2: Net-(D7-Pad1) -> GND
- R2 pad 1: /Power/Battery + -> /Power/+5V (INPUT PROTECTED)
- R2 pad 2: Net-(C3-Pad2) -> Net-(C1-Pad1)
- R3 pad 1: Net-(C3-Pad2) -> Net-(D2-Pad1)
- R4 pad 1: /microcontroller_interfacing/+5V -> /PA4
- R4 pad 2: /PA4 -> GND
- R5 pad 1: /PA4 -> VDD
- R5 pad 2: GND -> /PB8
- R6 pad 1: Net-(D4-Pad1) -> VDD
- R6 pad 2: GND -> /PB7
- R7 pad 1: VDD -> Net-(D6-Pad1)
- R7 pad 2: /PB8 -> Net-(R7-Pad2)
- R8 pad 1: VDD -> Net-(R8-Pad1)
- R8 pad 2: /PB7 -> GND
- R9 pad 2: Net-(D5-Pad1) -> Net-(C3-Pad2)
- TP5 pad 1: /Sensing/Temperature_Sensor/Vdd -> /PB1
- U1 pad 1: Net-(C2-Pad1) -> GND
- U1 pad 2: unconnected-(U1-Pad2) -> Net-(R8-Pad1)
- U1 pad 4: GND -> Net-(C1-Pad1)
- U1 pad 5: unconnected-(U1-Pad5) -> /Power/Battery +
- U1 pad 6: unconnected-(U1-Pad6) -> Net-(R3-Pad2)
- U1 pad 7: Net-(C3-Pad2) -> Net-(R7-Pad2)
- U1 pad 8: /Power/+5V jumped -> Net-(C1-Pad1)
- U2 pad 1: GND -> Net-(Q2-Pad1)
- U2 pad 2: VDD -> Net-(R13-Pad1)
- U2 pad 3: /Power/+5V (protected_jumped) -> Net-(Q3-Pad1)
- U3 pad 4: /microcontroller_interfacing/+5V -> Net-(C7-Pad1)
- U3 pad 5: Net-(JP7-Pad2) -> Net-(JP6-Pad2)
- U3 pad 6: Net-(JP8-Pad2) -> Net-(JP7-Pad2)
- U4 pad 1: /microcontroller_interfacing/+5V -> /microcontroller_interfacing/USB_Detect
- U5 pad 5: Net-(JP9-Pad1) -> Net-(JP8-Pad1)
- U5 pad 6: Net-(JP10-Pad1) -> Net-(JP9-Pad1)
- U6 pad 1: Net-(Q2-Pad2) -> GND
- U6 pad 2: Net-(D5-Pad1) -> VDD
- U6 pad 3: Net-(R10-Pad2) -> /Power/+5V (protected_jumped)
- U7 pad 1: unconnected-(U7-Pad1) -> /PB5
- U7 pad 10: /Sensing/Proximity_Sensor/VCC -> Net-(C10-Pad1)
- U7 pad 4: /PB0 -> /PB4
- U7 pad 8: /Sensing/Proximity_Sensor/VCC -> Net-(C10-Pad1)
- U8 pad 1: /Sensing/Temperature_Sensor/Vdd -> Net-(C12-Pad1)
- U8 pad 2: /PB4 -> /PB1
Routing:
- net VDD: track 201.8 -> 10.2 mm, vias 3 -> 0
- net /PB8: track 185.4 -> 10.2 mm, vias 7 -> 0
- net /microcontroller_interfacing/+5V: track 159.5 -> 0.00 mm
- net /PB7: track 162.7 -> 10.2 mm, vias 4 -> 0
- net /Power/Battery +: track 150.6 -> 2.55 mm, vias 2 -> 0
- net /PA4: track 149.7 -> 10.2 mm, vias 3 -> 0
- net /PB4: track 139.1 -> 10.3 mm, vias 2 -> 0
- net /PA10: track 103.0 -> 10.2 mm, vias 4 -> 0
- net /PA9: track 100.0 -> 10.2 mm, vias 2 -> 0
- net /Power/+5V (REVERSE PROTECTED): track 49.9 -> 0.00 mm, vias 2 -> 0
- net GND: track 85.4 -> 50.9 mm, vias 14 -> 0
- net /PB1: track 43.9 -> 10.2 mm
- net /PB0: track 43.8 -> 10.2 mm, vias 2 -> 0
- net /Sensing/Proximity_Sensor/VCC: track 31.7 -> 0.00 mm
- net Net-(C8-Pad1): track 29.1 -> 0.00 mm, vias 2 -> 0
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
Commit message: Final Schematic changes
Changed lines of the file:
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@@
     (property "Sheetfile" "power.kicad_sch")
     (property "Sheetname" "Power")
-    (attr smd exclude_from_pos_files)
+    (attr smd exclude_from_pos_files exclude_from_bom)
     (fp_text reference "BT1" (at 0 -0.5 unlocked) (layer "F.SilkS")
       (effects (font (size 1 1) (thickness 0.15)))
@@
     (property "Sheetfile" "sensing.kicad_sch")
     (property "Sheetname" "Sensing")
-    (attr exclude_from_pos_files)
+    (attr exclude_from_pos_files exclude_from_bom)
     (fp_text reference "JP5" (at 0 -1.85 90) (layer "F.SilkS")
       (effects (font (size 1 1) (thickness 0.15)))
@@
     (property "Sheetfile" "microcontroller_interfacing.kicad_sch")
     (property "Sheetname" "microcontroller_interfacing")
-    (attr exclude_from_pos_files)
+    (attr exclude_from_pos_files exclude_from_bom)
     (fp_text reference "JP7" (at 0 -1.8) (layer "F.SilkS")
       (effects (font (size 1 1) (thickness 0.15)))
@@
     (property "Sheetfile" "microcontroller_interfacing.kicad_sch")
     (property "Sheetname" "microcontroller_interfacing")
-    (attr exclude_from_pos_files)
+    (attr exclude_from_pos_files exclude_from_bom)
     (fp_text reference "JP8" (at 0 -1.8) (layer "F.SilkS")
       (effects (font (size 1 1) (thickness 0.15)))
@@
     (property "Sheetfile" "microcontroller_interfacing.kicad_sch")
     (property "Sheetname" "microcontroller_interfacing")
-    (attr exclude_from_pos_files)
+    (attr exclude_from_pos_files exclude_from_bom)
     (fp_text reference "JP6" (at 0 -1.8 90) (layer "F.SilkS")
       (effects (font (size 1 1) (thickness 0.15)))
@@
     (property "Sheetfile" "microcontroller_interfacing.kicad_sch")
     (property "Sheetname" "microcontroller_interfacing")
-    (attr exclude_from_pos_files)
+    (attr exclude_from_pos_files exclude_from_bom)
     (fp_text reference "JP9" (at 0.25 -2.1 90) (layer "F.SilkS")
       (effects (font (size 1 1) (thickness 0.15)))
@@
     (property "Sheetfile" "main.kicad_sch")
     (property "Sheetname" "")
-    (attr through_hole exclude_from_pos_files)
+    (attr through_hole exclude_from_pos_files exclude_from_bom)
     (fp_text reference "J3" (at 0 -2.33 -90) (layer "F.SilkS")
       (effects (font (size 1 1) (thickness 0.15)))
@@
     (property "Sheetfile" "main.kicad_sch")
     (property "Sheetname" "")
-    (attr through_hole exclude_from_pos_files)
+    (attr through_hole exclude_from_pos_files exclude_from_bom)
     (fp_text reference "J2" (at 0 -2.33 90) (layer "F.SilkS")
       (effects (font (size 1 1) (thickness 0.15)))
@@
     (property "Sheetfile" "power.kicad_sch")
     (property "Sheetname" "Power")
-    (attr exclude_from_pos_files)
+    (attr exclude_from_pos_files exclude_from_bom)
     (fp_text reference "JP2" (at -0.15 2) (layer "F.SilkS")
       (effects (font (size 1 1) (thickness 0.15)))
@@
     (property "Sheetfile" "main.kicad_sch")
     (property "Sheetname" "")
-    (attr through_hole exclude_from_pos_files)
+    (attr through_hole exclude_from_pos_files exclude_from_bom)
     (fp_text reference "J5" (at 0 -2.33 90) (layer "F.SilkS")
       (effects (font (size 1 1) (thickness 0.15)))
@@
     (property "Sheetfile" "main.kicad_sch")
     (property "Sheetname" "")
-    (attr through_hole exclude_from_pos_files)
+    (attr through_hole exclude_from_pos_files exclude_from_bom)
     (fp_text reference "J4" (at 0 -2.33 -90) (layer "F.SilkS")
       (effects (font (size 1 1) (thickness 0.15)))
@@
     (property "Sheetfile" "main.kicad_sch")
     (property "Sheetname" "")
-    (attr through_hole exclude_from_pos_files)
+    (attr through_hole exclude_from_pos_files exclude_from_bom)
     (fp_text reference "J1" (at 0 -2.33 90) (layer "F.SilkS")
       (effects (font (size 1 1) (thickness 0.15)))
@@
     (property "Sheetfile" "power.kicad_sch")
     (property "Sheetname" "Power")
-    (attr exclude_from_pos_files)
+    (attr exclude_from_pos_files exclude_from_bom)
     (fp_text reference "JP3" (at -0.1 -2.25) (layer "F.SilkS")
       (effects (font (size 1 1) (thickness 0.15)))
@@
     (property "Sheetfile" "power.kicad_sch")
     (property "Sheetname" "Power")
-    (attr exclude_from_pos_files)
+    (attr exclude_from_pos_files exclude_from_bom)
     (fp_text reference "JP4" (at 1.4 1.8 -270) (layer "F.SilkS")
       (effects (font (size 1 1) (thickness 0.15)))
@@
     (property "Sheetfile" "power.kicad_sch")
     (property "Sheetname" "Power")
-    (attr exclude_from_pos_files)
+    (attr exclude_from_pos_files exclude_from_bom)
     (fp_text reference "TP2" (at 0 1.448) (layer "B.SilkS")
       (effects (font (size 1 1) (thickness 0.15)) (justify mirror))
@@
     (property "Sheetfile" "power.kicad_sch")
     (property "Sheetname" "Power")
-    (attr exclude_from_pos_files)
+    (attr exclude_from_pos_files exclude_from_bom)
     (fp_text reference "TP1" (at 0 1.448) (layer "B.SilkS")
       (effects (font (size 1 1) (thickness 0.15)) (justify mirror))
@@
     (property "Sheetfile" "temperature_sensor.kicad_sch")
     (property "Sheetname" "Temperature_Sensor")
-    (attr exclude_from_pos_files)
+    (attr exclude_from_pos_files exclude_from_bom)
     (fp_text reference "TP5" (at 0 1.448) (layer "B.SilkS")
       (effects (font (size 1 1) (thickness 0.15)) (justify mirror))
@@
     (property "Sheetfile" "microcontroller_interfacing.kicad_sch")
     (property "Sheetname" "microcontroller_interfacing")
-    (attr exclude_from_pos_files)
+    (attr exclude_from_pos_files exclude_from_bom)
     (fp_text reference "TP3" (at 0 1.448) (layer "B.SilkS")
       (effects (font (size 1 1) (thickness 0.15)) (justify mirror))
@@
     (effects (font (size 0.7 0.7) (thickness 0.1)) (justify mirror))
   )
-  (gr_text "Proximity and\nTemperature HAT" (at 219.65 86.45) (layer "F.SilkS")
+  (gr_text "Proximity and\nTemperature HAT" (at 250.4 60.225) (layer "F.SilkS")
     (effects (font (size 2 2) (thickness 0.25)))
   )
@@
     (effects (font (size 1 1) (thickness 0.15)))
   )
-  (gr_text "Heather, Kelvin, Noah\nGroup 5" (at 218.95 78.65) (layer "F.SilkS")
+  (gr_text "Heather, Kelvin, Noah\nGroup 5" (at 250.6 52.1) (layer "F.SilkS")
     (effects (font (size 2 2) (thickness 0.25)))
   )

Commit message: PCB changes
Parts:
- Q2, Q3: value AO3401A -> 2N7002
Changed lines of the file:
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@@
     (property "Sheetfile" "power.kicad_sch")
     (property "Sheetname" "Power")
-    (attr smd exclude_from_pos_files exclude_from_bom)
+    (attr smd exclude_from_pos_files)
     (fp_text reference "BT1" (at 0 -0.5 unlocked) (layer "F.SilkS")
       (effects (font (size 1 1) (thickness 0.15)))
@@
     (property "Sheetfile" "sensing.kicad_sch")
     (property "Sheetname" "Sensing")
-    (attr exclude_from_pos_files exclude_from_bom)
+    (attr exclude_from_pos_files)
     (fp_text reference "JP5" (at 0 -1.85 90) (layer "F.SilkS")
       (effects (font (size 1 1) (thickness 0.15)))
@@
     (property "Sheetfile" "microcontroller_interfacing.kicad_sch")
     (property "Sheetname" "microcontroller_interfacing")
-    (attr exclude_from_pos_files exclude_from_bom)
+    (attr exclude_from_pos_files)
     (fp_text reference "JP7" (at 0 -1.8) (layer "F.SilkS")
       (effects (font (size 1 1) (thickness 0.15)))
@@
     (descr "SOT, 3 Pin (https://www.jedec.org/system/files/docs/to-236h.pdf variant AB), generated with kicad-footprint-generator ipc_gullwing_generator.py")
     (tags "SOT TO_SOT_SMD")
-    (property "JLC Part #" "C15127")
-    (property "LCSC" "C15127")
+    (property "JLC Part #" "C8545")
+    (property "LCSC" "C8545")
     (property "Sheetfile" "power.kicad_sch")
     (property "Sheetname" "Power")
@@
       (effects (font (size 1 1) (thickness 0.15)))
     )
-    (fp_text value "AO3401A" (at 0 2.4 180) (layer "F.Fab")
+    (fp_text value "2N7002" (at 0 2.4 180) (layer "F.Fab")
       (effects (font (size 1 1) (thickness 0.15)))
     )
@@
     (property "Sheetfile" "microcontroller_interfacing.kicad_sch")
     (property "Sheetname" "microcontroller_interfacing")
-    (attr exclude_from_pos_files exclude_from_bom)
+    (attr exclude_from_pos_files)
     (fp_text reference "JP8" (at 0 -1.8) (layer "F.SilkS")
       (effects (font (size 1 1) (thickness 0.15)))
@@
     (property "Sheetfile" "microcontroller_interfacing.kicad_sch")
     (property "Sheetname" "microcontroller_interfacing")
-    (attr exclude_from_pos_files exclude_from_bom)
+    (attr exclude_from_pos_files)
     (fp_text reference "JP6" (at 0 -1.8 90) (layer "F.SilkS")
       (effects (font (size 1 1) (thickness 0.15)))
@@
     (property "Sheetfile" "microcontroller_interfacing.kicad_sch")
     (property "Sheetname" "microcontroller_interfacing")
-    (attr exclude_from_pos_files exclude_from_bom)
+    (attr exclude_from_pos_files)
     (fp_text reference "JP9" (at 0.25 -2.1 90) (layer "F.SilkS")
       (effects (font (size 1 1) (thickness 0.15)))
@@
     (property "Sheetfile" "main.kicad_sch")
     (property "Sheetname" "")
-    (attr through_hole exclude_from_pos_files exclude_from_bom)
+    (attr through_hole exclude_from_pos_files)
     (fp_text reference "J3" (at 0 -2.33 -90) (layer "F.SilkS")
       (effects (font (size 1 1) (thickness 0.15)))
@@
     (property "Sheetfile" "main.kicad_sch")
     (property "Sheetname" "")
-    (attr through_hole exclude_from_pos_files exclude_from_bom)
+    (attr through_hole exclude_from_pos_files)
     (fp_text reference "J2" (at 0 -2.33 90) (layer "F.SilkS")
       (effects (font (size 1 1) (thickness 0.15)))
@@
     (property "Sheetfile" "power.kicad_sch")
     (property "Sheetname" "Power")
-    (attr exclude_from_pos_files exclude_from_bom)
+    (attr exclude_from_pos_files)
     (fp_text reference "JP2" (at -0.15 2) (layer "F.SilkS")
       (effects (font (size 1 1) (thickness 0.15)))
@@
     (descr "SOT, 3 Pin (https://www.jedec.org/system/files/docs/to-236h.pdf variant AB), generated with kicad-footprint-generator ipc_gullwing_generator.py")
     (tags "SOT TO_SOT_SMD")
-    (property "JLC Part #" "C15127")
-    (property "LCSC" "C15127")
+    (property "JLC Part #" "C8545")
+    (property "LCSC" "C8545")
     (property "Sheetfile" "power.kicad_sch")
     (property "Sheetname" "Power")
@@
       (effects (font (size 1 1) (thickness 0.15)))
     )
-    (fp_text value "AO3401A" (at 0 2.4) (layer "F.Fab")
+    (fp_text value "2N7002" (at 0 2.4) (layer "F.Fab")
       (effects (font (size 1 1) (thickness 0.15)))
     )
@@
     (property "Sheetfile" "main.kicad_sch")
     (property "Sheetname" "")
-    (attr through_hole exclude_from_pos_files exclude_from_bom)
+    (attr through_hole exclude_from_pos_files)
     (fp_text reference "J5" (at 0 -2.33 90) (layer "F.SilkS")
       (effects (font (size 1 1) (thickness 0.15)))
@@
     (property "Sheetfile" "main.kicad_sch")
     (property "Sheetname" "")
-    (attr through_hole exclude_from_pos_files exclude_from_bom)
+    (attr through_hole exclude_from_pos_files)
     (fp_text reference "J4" (at 0 -2.33 -90) (layer "F.SilkS")
       (effects (font (size 1 1) (thickness 0.15)))
@@
     (property "Sheetfile" "main.kicad_sch")
     (property "Sheetname" "")
-    (attr through_hole exclude_from_pos_files exclude_from_bom)
+    (attr through_hole exclude_from_pos_files)
     (fp_text reference "J1" (at 0 -2.33 90) (layer "F.SilkS")
       (effects (font (size 1 1) (thickness 0.15)))
@@
     (property "Sheetfile" "power.kicad_sch")
     (property "Sheetname" "Power")
-    (attr exclude_from_pos_files exclude_from_bom)
+    (attr exclude_from_pos_files)
     (fp_text reference "JP3" (at -0.1 -2.25) (layer "F.SilkS")
       (effects (font (size 1 1) (thickness 0.15)))
@@
     (property "Sheetfile" "power.kicad_sch")
     (property "Sheetname" "Power")
-    (attr exclude_from_pos_files exclude_from_bom)
+    (attr exclude_from_pos_files)
     (fp_text reference "JP4" (at 1.4 1.8 -270) (layer "F.SilkS")
       (effects (font (size 1 1) (thickness 0.15)))
@@
     (property "Sheetfile" "power.kicad_sch")
     (property "Sheetname" "Power")
-    (attr exclude_from_pos_files exclude_from_bom)
+    (attr exclude_from_pos_files)
     (fp_text reference "TP2" (at 0 1.448) (layer "B.SilkS")
       (effects (font (size 1 1) (thickness 0.15)) (justify mirror))
@@
     (property "Sheetfile" "power.kicad_sch")
     (property "Sheetname" "Power")
-    (attr exclude_from_pos_files exclude_from_bom)
+    (attr exclude_from_pos_files)
     (fp_text reference "TP1" (at 0 1.448) (layer "B.SilkS")
       (effects (font (size 1 1) (thickness 0.15)) (justify mirror))
@@
     (property "Sheetfile" "temperature_sensor.kicad_sch")
     (property "Sheetname" "Temperature_Sensor")
-    (attr exclude_from_pos_files exclude_from_bom)
+    (attr exclude_from_pos_files)
     (fp_text reference "TP5" (at 0 1.448) (layer "B.SilkS")
       (effects (font (size 1 1) (thickness 0.15)) (justify mirror))
@@
     (property "Sheetfile" "microcontroller_interfacing.kicad_sch")
     (property "Sheetname" "microcontroller_interfacing")
-    (attr exclude_from_pos_files exclude_from_bom)
+    (attr exclude_from_pos_files)
     (fp_text reference "TP3" (at 0 1.448) (layer "B.SilkS")
       (effects (font (size 1 1) (thickness 0.15)) (justify mirror))

Commit message: Final PCB design
Parts:
- moved R10 104.7 mm to (99.3, 106.5)
- moved R11 104.4 mm to (92.9, 109.8)
- moved JP6 98.8 mm to (172.2, 88.2), turned to 180 degrees
- moved R13 94.0 mm to (149.4, 152.9), turned to 180 degrees
- moved G*** 83.6 mm to (122.5, 90.1)
- moved R5 74.6 mm to (144.4, 110.3)
- moved C3 67.1 mm to (160.2, 153.0), turned to 90 degrees
- moved TP2 61.0 mm to (168.9, 131.3)
- moved Q3 60.9 mm to (152.0, 159.7), turned to -90 degrees
- moved C6 59.2 mm to (166.0, 81.1), turned to -90 degrees
- moved D2 58.3 mm to (173.9, 130.9)
- moved C8 54.5 mm to (173.9, 81.0), turned to -90 degrees
- moved R1 53.9 mm to (165.8, 110.0)
- moved Q2 53.7 mm to (158.7, 159.7), turned to -90 degrees
- moved U2 53.5 mm to (154.8, 153.8)
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Routing:
- net /PB8: track 10.2 -> 152.3 mm, vias 0 -> 5
- net /PB7: track 10.2 -> 136.3 mm, vias 0 -> 5
- net /PB4: track 10.3 -> 133.6 mm, vias 0 -> 1
- net /PA4: track 10.2 -> 133.3 mm, vias 0 -> 4
- net VDD: track 10.2 -> 128.0 mm, vias 0 -> 3
- net Net-(BT1-Pad2): track 0.00 -> 85.2 mm, vias 0 -> 2
- net /PA9: track 10.2 -> 92.4 mm, vias 0 -> 1
- net /microcontroller_interfacing/+5V: track 0.00 -> 79.6 mm, vias 0 -> 3
- net /PA10: track 10.2 -> 88.5 mm, vias 0 -> 2
- net /PB5: track 10.2 -> 83.8 mm, vias 0 -> 5
- net Net-(C1-Pad1): track 0.00 -> 45.7 mm, vias 0 -> 4
- net Net-(C10-Pad1): track 0.00 -> 41.0 mm
- net /Power/Battery +: track 2.55 -> 41.6 mm
- net /PB1: track 10.2 -> 41.9 mm, vias 0 -> 1
- net GND: track 50.9 -> 80.6 mm, vias 0 -> 10
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Other:
- board text added: "Ver 2 https://gitlab.com/wmbhea001 /eee088f-group-5"
- board text removed: "TempVcc"
- board text removed: "UVCutPro"
- board text removed: "Ver 1 https://gitlab.com/wmbhea001/eee088f-group-5"
